File: angled-ten-sipm-carrier/single-sipm.kicad_sch (KiCad schematic)
At the start: 2 parts, among them U6 MICROFC-60035-SMT-TR1

Commit message: update sipm board pre-em
Connections:
- no-connect marks 1 -> 0
Changed lines of the file:
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@@
 		(color 0 0 0 0)
-	)
-	(no_connect
-		(at 64.77 40.64)
 	)
 	(wire
@@
 		(shape input)
 		(at 45.72 25.4 180)
-		(fields_autoplaced yes)
 		(effects
 			(font
@@
 		(shape output)
 		(at 54.61 55.88 0)
-		(fields_autoplaced yes)
 		(effects
 			(font
@@
 		(pin "3"
 		)
-		(pin "2"
-		)
 		(instances

Commit message: broadcom board v1
Parts:
- removed U6: MICROFC-60035-SMT-TR1, Library:XDCR_MICROFC-60035-SMT-TR1, symbol Library:MICROFC-60035-SMT-TR1
- added D1: AFBR-S4N66P014M, Library:AFBRS4N66P014M, symbol Library:AFBR-S4N66P014M
- renumbered C13 to C10
Connections:
- net anode (out): now also D1.B2 (anode), D1.B3 (anode), D1.C2 (anode), D1.C3 (anode)
- net bias: now also D1.A1 (cathode), D1.A4 (cathode), D1.D1 (cathode), D1.D4 (cathode)

Commit message: touch up broadcom
Parts:
- C10: value 10p -> 10n
Changed lines of the file:
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@@
 			)
 		)
-		(property "Value" "10p"
+		(property "Value" "10n"
 			(at 55.88 20.32 90)
 			(effects
