File: fc-board/fc-board.kicad_pcb (KiCad board)
At the start: 4 copper layers, 95.9 x 90.2 mm, 84 parts, among them J1 ESQ-125-14-G-D, J2 MSXS-08PFFR-SF7002, J3 M80-5322042, J4 M80-5102622, J5 SMA-J-P-X-ST-TH1, J6 10067847-001RLF, U1 749023310, U2 74LVC1G07SE-7, U3 ADS1015BQDGSRQ1, U4 PCT2075TP_147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

Commit message: Added test points to I2C lines
Parts:
- added TP3: SDA, fc-board:TestPoint_THTPad_D2.0mm_Drill1.0mm_JLCrules, F.Cu at (103.0, 35.0)
- added TP4: SCL, fc-board:TestPoint_THTPad_D2.0mm_Drill1.0mm_JLCrules, F.Cu at (106.5, 35.0)
Routing:
- net /gpio/I2C1_SCL: track 139.2 -> 148.0 mm
- net /gpio/I2C1_SDA: track 144.3 -> 147.0 mm
