File: fc-board/gpio-hispeed.kicad_sch (KiCad schematic)
At the start: 6 parts, among them J7 685119134923, U9 RT9742SNGV

Commit message: FC board updates
Parts:
- removed C19, C20: 100n, Capacitor_SMD:C_1206_3216Metric, symbol Device:C_Small
- removed J7: 685119134923, fc-board:685119134923, symbol fc-board:685119134923
- removed JP13: OTG TO GND, Jumper:SolderJumper-2_P1.3mm_Open_Pad1.0x1.5mm, symbol Jumper:SolderJumper_2_Open
- removed U9: RT9742SNGV, fc-board:RT9742SNGV, symbol fc-board:RT9742SNGV
- added JP5: OTG TO GND, Jumper:SolderJumper-2_P1.3mm_Open_Pad1.0x1.5mm, symbol Jumper:SolderJumper_2_Open
Connections:
- net GND: now also JP5.2 (B)
- net PCIE_CLK_nREQ: now reaches Module1.102 (PCIe_CLK_nREQ)
- net PCIE_nRST: now reaches Module1.109 (PCIe_nRST)
- net PCIE_CLK_P: now reaches Module1.110 (PCIe_CLK_P)
- net PCIE_CLK_N: now reaches Module1.112 (PCIe_CLK_N)
- net PCIE_RX_P: now reaches Module1.116 (PCIe_RX_P)
- net PCIE_RX_N: now reaches Module1.118 (PCIe_RX_N)
- net PCIE_TX_P: now reaches Module1.122 (PCIe_TX_P)
- net PCIE_TX_N: now reaches Module1.124 (PCIe_TX_N)
- net HDMI0_CEC: no longer names the net of Module1.151 (HDMI0_CEC)
- net HDMI0_CK_N: no longer names the net of Module1.190 (HDMI0_CLK_N)
- net HDMI0_CK_P: no longer names the net of Module1.188 (HDMI0_CLK_P)
- net HDMI0_D0_N: no longer names the net of Module1.184 (HDMI0_TX0_N)
- net HDMI0_D0_P: no longer names the net of Module1.182 (HDMI0_TX0_P)
- net HDMI0_D1_N: no longer names the net of Module1.178 (HDMI0_TX1_N)
- net HDMI0_D1_P: no longer names the net of Module1.176 (HDMI0_TX1_P)
- net HDMI0_D2_N: no longer names the net of Module1.172 (HDMI0_TX2_N)
- net HDMI0_D2_P: no longer names the net of Module1.170 (HDMI0_TX2_P)
- net HDMI0_HOTPLUG: no longer names the net of Module1.153 (HDMI0_HOTPLUG)
- net HDMI0_SCL: no longer names the net of Module1.200 (HDMI0_SCL)
- net HDMI0_SDA: no longer names the net of Module1.199 (HDMI0_SDA)
- net USB2_N: no longer names the net of Module1.103 (USB2_N)
- net USB2_P: no longer names the net of Module1.105 (USB2_P)
- net USB_OTG_ID: no longer names the net of Module1.101 (USB_OTG_ID)
- net USB_OTG_ID: now also JP5.1 (A)
- no-connect marks 55 -> 62
Other:
- added sheet pcie-ethernet (pcie-ethernet.kicad_sch)
- note removed: "Copied from the IO board"
- moved on the sheet: Module1B

Commit message: Finished routing; cleaned library
Parts:
- renumbered JP5 to JP7
Connections:
- net USB_N: now reaches Module1.103 (USB2_N)
- net USB_P: now reaches Module1.105 (USB2_P)
- no-connect marks 62 -> 60
Other:
- sheet pcie-ethernet ports: added PCIE_CLK_N, PCIE_RX_N, PCIE_TX_N; removed PCIE_CLK_M, PCIE_RX_M, PCIE_TX_M
Changed lines of the file:
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@@
 	(title_block
 		(title "CM4 Hi-speed Serial")
-		(date "2024-09-12")
+		(date "2025-10-17")
 		(rev "0.1")
 	)
@@
 	)
 	(no_connect
-		(at 110.49 43.18)
-	)
-	(no_connect
 		(at 110.49 66.04)
 	)
@@
 		(at 49.53 142.24)
 	)
-	(no_connect
-		(at 110.49 40.64)
-	)
 	(wire
 		(pts
@@
 	(wire
 		(pts
+			(xy 110.49 43.18) (xy 130.81 43.18)
+		)
+		(stroke
+			(width 0)
+			(type default)
+		)
+	)
+	(wire
+		(pts
 			(xy 142.24 64.77) (xy 161.29 64.77)
 		)
@@
 		(pts
 			(xy 110.49 68.58) (xy 111.76 68.58)
+		)
+		(stroke
+			(width 0)
+			(type default)
+		)
+	)
+	(wire
+		(pts
+			(xy 110.49 40.64) (xy 130.81 40.64)
 		)
 		(stroke
@@
 		)
 	)
+	(hierarchical_label "USB_N"
+		(shape output)
+		(at 130.81 40.64 0)
+		(effects
+			(font
+				(size 1.27 1.27)
+			)
+			(justify left)
+		)
+	)
 	(hierarchical_label "Y4-"
 		(shape output)
@@
 		(shape output)
 		(at 199.39 73.66 0)
+		(effects
+			(font
+				(size 1.27 1.27)
+			)
+			(justify left)
+		)
+	)
+	(hierarchical_label "USB_P"
+		(shape output)
+		(at 130.81 43.18 0)
 		(effects
 			(font
@@
 		(dnp no)
 		(fields_autoplaced yes)
-		(property "Reference" "#PWR023"
+		(property "Reference" "#PWR027"
 			(at 116.84 21.59 0)
 			(effects
@@
 			(project ""
 				(path "/14bbabed-904f-4efc-8ba4-be00e59385c4/edd7e4f6-7524-424d-ae74-0eda33819a09"
-					(reference "#PWR023")
+					(reference "#PWR027")
 					(unit 1)
 				)
@@
 		(dnp no)
 		(fields_autoplaced yes)
-		(property "Reference" "#PWR021"
+		(property "Reference" "#PWR025"
 			(at 48.26 179.07 0)
 			(effects
@@
 			(project "fc-board"
 				(path "/14bbabed-904f-4efc-8ba4-be00e59385c4/edd7e4f6-7524-424d-ae74-0eda33819a09"
-					(reference "#PWR021")
+					(reference "#PWR025")
 					(unit 1)
 				)
@@
 		(dnp no)
 		(fields_autoplaced yes)
-		(property "Reference" "#PWR022"
+		(property "Reference" "#PWR026"
 			(at 111.76 179.07 0)
 			(effects
@@
 			(project "fc-board"
 				(path "/14bbabed-904f-4efc-8ba4-be00e59385c4/edd7e4f6-7524-424d-ae74-0eda33819a09"
-					(reference "#PWR022")
+					(reference "#PWR026")
 					(unit 1)
 				)
@@
 		(dnp no)
 		(fields_autoplaced yes)
-		(property "Reference" "JP5"
+		(property "Reference" "JP7"
 			(at 119.38 30.4799 90)
 			(effects
@@
 			(project ""
 				(path "/14bbabed-904f-4efc-8ba4-be00e59385c4/edd7e4f6-7524-424d-ae74-0eda33819a09"
-					(reference "JP5")
+					(reference "JP7")
 					(unit 1)
 				)
@@
 			)
 		)
-		(pin "PCIE_RX_M" output
-			(at 162.56 78.74 180)
-			(effects
-				(font
-					(size 1.27 1.27)
-				)
-				(justify left)
-			)
-		)
 		(pin "TRD-" output
 			(at 196.85 86.36 0)
@@
 			)
 		)
-		(pin "PCIE_TX_M" output
-			(at 162.56 73.66 180)
-			(effects
-				(font
-					(size 1.27 1.27)
-				)
-				(justify left)
-			)
-		)
 		(pin "DUPLEX_LED" output
 			(at 196.85 92.71 0)
@@
 			)
 		)
-		(pin "PCIE_CLK_M" output
+		(pin "PCIE_RX_N" output
+			(at 162.56 78.74 180)
+			(effects
+				(font
+					(size 1.27 1.27)
+				)
+				(justify left)
+			)
+		)
+		(pin "PCIE_TX_N" output
+			(at 162.56 73.66 180)
+			(effects
+				(font
+					(size 1.27 1.27)
+				)
+				(justify left)
+			)
+		)
+		(pin "PCIE_CLK_N" output
 			(at 162.56 85.09 180)
 			(effects
