File: fc-board/i2c-hub.kicad_sch (KiCad schematic)
At the start: 54 parts, among them U5 PCT2075TP_147, U6 MAX11617EEE+, U7 DS3231M+TRL, U8 TLV9004QPWRQ1, U9 ADS122C04IPWR

Commit message: Updated RJ45 jack
Parts:
- renumbered C12 to C10, C13 to C11, C14 to C12, C15 to C13, C16 to C14, C8 to C6, C9 to C7, C10 to C8, C11 to C9

Commit message: Assigned part numbers to everything, replaced ethernet jack
Parts:
- C6: value 1u -> 0.1u
- R18, R26: value 71.4k -> 71.5k
- R19, R30: value 161.3k -> 162k
- R20, R27, R35, R36: value 250k -> 249k
- R22, R23: value 9.8k -> 10k
- R32: value 5k -> 4.99k
- renumbered JP8 to JP7

Commit message: fix stupid merge issue
Parts:
- BT1: now left out of the parts list
- R14: renamed from R15; value 10k -> 1k
- R21: renamed from R22; value 10k -> 4.87k
- R22: renamed from R23; value 10k -> 4.87k
- TP10: renamed from TP12; symbol Connector:TestPoint -> fc-board:TestPoint; now left out of the parts list
- TP11: renamed from TP13; symbol Connector:TestPoint -> fc-board:TestPoint; now left out of the parts list
- TP12: renamed from TP14; symbol Connector:TestPoint -> fc-board:TestPoint; now left out of the parts list
- TP9: renamed from TP11; symbol Connector:TestPoint -> fc-board:TestPoint; now left out of the parts list
- renumbered JP7 to JP10, R13 to R12, R14 to R13, R16 to R15, R17 to R16, R18 to R17, R19 to R18, R20 to R19, R21 to R20, R24 to R23, R25 to R24, R26 to R25, R27 to R26, R28 to R27, R29 to R28, R30 to R29, R31 to R30, R32 to R31, R33 to R32, R34 to R33, R35 to R34, R36 to R35, U5 to U2, U6 to U3, U7 to U4, U8 to U5, U9 to U6
Connections:
- net ADS_RESET is gone; now on net 3.3V_IN: U6.3 (RESET)
- net +5V_CM4: now also R14.1
- net 3.3V_IN: no longer R14.1
Other:
- note added: "These two resistors form the second half of the voltage divider started on the bias board; with 150k and 4.87k, our bias ranges from 0.88 to 1.51 V (corresponding to 28 to 48 V) across the digipot range."
- note removed: "These two resistors form the second half of the voltage divider started on the bias board; with 150k and 7k, our bias ranges from 1.427 to 2.176 V (corresponding to 32.4 to 48.8 V) across the digipot range. This is then added on the 1.024 V reference voltage."
- note removed: "Will we have a coincell battery?"
- moved on the sheet: BT1, C7, JP10, R13, R14, TP10, TP11, TP12, U4
