File: emmc-tester/emmc-tester.kicad_pcb (KiCad board)
At the start: 2 copper layers, 30.5 x 20.2 mm, 10 parts, among them J1 Micro_SD_Card

Commit message: thickness and mounting holes
Parts:
- added H1: MountingHole, MountingHole:MountingHole_3.2mm_M3, F.Cu at (85.2, 25.0)
- added H2: MountingHole, MountingHole:MountingHole_3.2mm_M3, F.Cu at (85.8, 39.8)
- added H3: MountingHole, MountingHole:MountingHole_3.2mm_M3, F.Cu at (62.8, 25.2)
- moved CVccq1 1.64 mm to (85.2, 35.1), turned to 0 degrees
Routing:
- net GND: vias 48 -> 39
