File: lvps-toggles-adapter/lvps-toggles-adapter.kicad_pcb (KiCad board)
At the start: 2 copper layers, 90 x 90 mm, 19 parts, among them J1 Toggle 1 in, J10 Toggle 2 out, J11 Toggle 3 out, J12 Toggle 4 out, J13 Bias/heat out, J14 bridgeports out, J15 Other heat connection, J2 Toggle 2 in, J3 Toggle 3 in, J4 Toggle 4 in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

Commit message: toggles adapter: cleanup
Connections:
- J11 pad 5: Net-(J11-Pin_5) -> GND
- J11 pad 6: Net-(J11-Pin_5) -> GND
- J11 pad 7: Net-(J11-Pin_5) -> GND
- J12 pad 5: Net-(J12-Pin_5) -> GND
- J12 pad 6: Net-(J12-Pin_5) -> GND
- J12 pad 7: Net-(J12-Pin_5) -> GND
- J8 pad 5: Net-(J8-Pin_5) -> GND
- J8 pad 6: Net-(J8-Pin_5) -> GND
- J8 pad 7: Net-(J8-Pin_5) -> GND
Routing:
- net Bridgeport 4 +5V: track 28.7 -> 29.5 mm
- net GND: vias 260 -> 262
- net /CHASSIS: vias 1484 -> 1501
Other:
- board text added: "BIAS/HEAT"
- board text added: "BRIDGEPORTS"
- board text added: "TOG1"
- board text added: "TOG2"
- board text added: "TOG3"
- board text added: "TOG4"
