File: lvps-toggles-swri/IMPISH Toggle Bd Sht4.kicad_sch (KiCad schematic)
At the start: 66 parts, among them J5 BCS-110-L-D-TE, J6 BCS-110-L-D-TE, Q13 MMBT3904Q, Q14 MMBT3906Q, Q15 ZXM61N02F, Q16 MMBT3904Q, Q17 MMBT3906Q, Q18 ZXM61N02F, Q19 MMBT3904Q, Q20 MMBT3906Q, Q21 ZXM61N02F, Q22 MMBT3904Q, Q23 MMBT3906Q, Q24 ZXM61N02F, U10 BSP452, U11 AP22804AW5-7, U12 AP22804AW5-7, U7 BSP452, U8 AP22804AW5-7, U9 AP22804AW5-7

Commit message: Power board updates (#7)
* toggles adapter board

The SwRI toggle output is in the wrong direction,
so we are adding an additional PCB to point the power
towards the side of the EPS box. We can route it with
cables and connectors instead of using the board-to-board
style interface.

* toggles adapter: cleanup

* toggles adapter: via stitching

* swri toggles: start one ground

* swri toggles: single ground pre stitching

* swri toggles: via stitching for gnd

* swri toggles: fix DRC and ERC errors

* swri lvps main: two layer board

* swri lvps main: fix cap models
Parts:
- removed R49, R50, R69, R70: 10, Resistor_SMD:R_0805_2012Metric_Pad1.20x1.40mm_HandSolder, symbol Device:R_Small_US
Connections:
- net Bridgeport GND is gone; now on net GND: C11.2, C13.2, C19.2, C21.2, J5.09, J5.10, J6.09, J6.10
- net Cremat GND is gone; now on net GND: J5.03, J5.04, J6.03, J6.04, Q13.2 (E), Q19.2 (E), R41.2, R46.2, R61.2, R66.2
- net GND1 is gone; now on net GND: C3.2, C4.2, U10.2 (GND), U11.2 (GND), U11.3 (FLG), U12.2 (GND), U12.3 (FLG), U7.2 (GND), U8.2 (GND), U8.3 (FLG), U9.2 (GND), U9.3 (FLG)
- net SiPM GND is gone; now on net GND: C12.2, C14.2, C20.2, C22.2, J5.13, J5.14, J6.13, J6.14, Q16.2 (E), Q22.2 (E), R51.2, R56.2, R71.2, R76.2
- net GND: now reaches J5.17, J5.18
- net GND: now also J5.19, J5.20, J6.17, J6.18, J6.19, J6.20
