File: lvps-toggles-swri/IMPISH Toggle Bd Sht5.kicad_sch (KiCad schematic)
At the start: 22 parts, among them J7 BCS-105-L-D-TE, J8 BCS-105-L-D-TE, Q25 MMBT3904Q, Q26 MMBT3906Q, Q27 ZXM61N02F, U13 BSP742T, U14 BSP452

Commit message: Power board updates (#7)
* toggles adapter board

The SwRI toggle output is in the wrong direction,
so we are adding an additional PCB to point the power
towards the side of the EPS box. We can route it with
cables and connectors instead of using the board-to-board
style interface.

* toggles adapter: cleanup

* toggles adapter: via stitching

* swri toggles: start one ground

* swri toggles: single ground pre stitching

* swri toggles: via stitching for gnd

* swri toggles: fix DRC and ERC errors

* swri lvps main: two layer board

* swri lvps main: fix cap models
Parts:
- removed R89, R90, R91, R92, R93: 10, Resistor_SMD:R_0805_2012Metric_Pad1.20x1.40mm_HandSolder, symbol Device:R_Small_US
Connections:
- net Bias GND is gone; now on net GND: J8.03, J8.04, Q25.2 (E), R81.2, R86.2
- net GND1 is gone; now on net GND: C5.2, C6.2, U13.1 (GND), U13.4 (NC), U14.2 (GND)
- net Heater GND is gone; now on net GND: J7.03, J7.04
- net GND: now reaches J8.09, J8.10
- net GND: now also J7.05, J7.06, J7.07, J7.08, J7.09, J7.10, J8.07, J8.08
