File: sipm-carrier-flight/single-sipm.kicad_sch (KiCad schematic)
At the start: 2 parts

Commit message: sipm board pre-production
- verify spcaing between SiPMs
- move silkscreens around so that they are not overlapping
- change footprints to be hand-solder type in case someone has to do that
- change values of some components to unify part list (e.g. any 100n are now 0.1u)
Parts:
- C10: footprint Capacitor_SMD:C_0805_2012Metric -> Capacitor_SMD:C_0805_2012Metric_Pad1.18x1.45mm_HandSolder
Changed lines of the file:
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@@
 			)
 		)
-		(property "Footprint" "Capacitor_SMD:C_0805_2012Metric"
+		(property "Footprint" "Capacitor_SMD:C_0805_2012Metric_Pad1.18x1.45mm_HandSolder"
 			(at 59.69 24.4348 0)
 			(effects
