File: bias-supply/gnd-stitching.kicad_sch (KiCad schematic)
At the start: 8 parts

Commit message: Updates for new bubba board
Parts:
- removed JP15, JP16, JP17, JP18, JP19: SolderJumper_2_Open, Resistor_SMD:R_1206_3216Metric, symbol Jumper:SolderJumper_2_Open
- added JP10, JP11, JP7, JP8, JP9: SolderJumper_2_Open, Resistor_SMD:R_1206_3216Metric, symbol Jumper:SolderJumper_2_Open
Connections:
- net GND: now also JP10.1 (A), JP10.2 (B), JP11.1 (A), JP11.2 (B), JP7.1 (A), JP7.2 (B), JP8.1 (A), JP8.2 (B), JP9.1 (A), JP9.2 (B)
Other:
- title: (none) -> Ground stitching

Commit message: Add fuses; change to coax; fixed I2C gnd
Parts:
- renumbered JP8 to JP10, JP9 to JP13, JP10 to JP14, JP13 to JP15, JP14 to JP16, JP7 to JP9
Changed lines of the file:
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@@
 		(on_board yes)
 		(dnp no)
-		(property "Reference" "#PWR055"
+		(property "Reference" "#PWR041"
 			(at 69.85 63.5 0)
 			(effects
@@
 			(project "bias-supply"
 				(path "/f3205b63-fc57-4ea3-95d4-2a447f249c30/2946e9e0-97c7-47f2-899e-bbb1d0cbea92"
-					(reference "#PWR055")
+					(reference "#PWR041")
 					(unit 1)
 				)
@@
 		(on_board yes)
 		(dnp no)
-		(property "Reference" "#PWR054"
+		(property "Reference" "#PWR040"
 			(at 69.85 53.34 0)
 			(effects
@@
 			(project "bias-supply"
 				(path "/f3205b63-fc57-4ea3-95d4-2a447f249c30/2946e9e0-97c7-47f2-899e-bbb1d0cbea92"
-					(reference "#PWR054")
+					(reference "#PWR040")
 					(unit 1)
 				)
@@
 		(on_board yes)
 		(dnp no)
-		(property "Reference" "#PWR046"
+		(property "Reference" "#PWR032"
 			(at 44.45 53.34 0)
 			(effects
@@
 			(project "bias-supply"
 				(path "/f3205b63-fc57-4ea3-95d4-2a447f249c30/2946e9e0-97c7-47f2-899e-bbb1d0cbea92"
-					(reference "#PWR046")
+					(reference "#PWR032")
 					(unit 1)
 				)
@@
 		(dnp no)
 		(fields_autoplaced yes)
-		(property "Reference" "JP8"
+		(property "Reference" "JP10"
 			(at 34.29 30.48 0)
 			(effects
@@
 			(project "bias-supply"
 				(path "/f3205b63-fc57-4ea3-95d4-2a447f249c30/2946e9e0-97c7-47f2-899e-bbb1d0cbea92"
-					(reference "JP8")
+					(reference "JP10")
 					(unit 1)
 				)
@@
 		(on_board yes)
 		(dnp no)
-		(property "Reference" "#PWR045"
+		(property "Reference" "#PWR031"
 			(at 44.45 36.83 0)
 			(effects
@@
 			(project "bias-supply"
 				(path "/f3205b63-fc57-4ea3-95d4-2a447f249c30/2946e9e0-97c7-47f2-899e-bbb1d0cbea92"
-					(reference "#PWR045")
+					(reference "#PWR031")
 					(unit 1)
 				)
@@
 		(dnp no)
 		(fields_autoplaced yes)
-		(property "Reference" "JP10"
+		(property "Reference" "JP14"
 			(at 59.69 30.48 0)
 			(effects
@@
 			(project "bias-supply"
 				(path "/f3205b63-fc57-4ea3-95d4-2a447f249c30/2946e9e0-97c7-47f2-899e-bbb1d0cbea92"
-					(reference "JP10")
+					(reference "JP14")
 					(unit 1)
 				)
@@
 		(on_board yes)
 		(dnp no)
-		(property "Reference" "#PWR051"
+		(property "Reference" "#PWR037"
 			(at 49.53 63.5 0)
 			(effects
@@
 			(project "bias-supply"
 				(path "/f3205b63-fc57-4ea3-95d4-2a447f249c30/2946e9e0-97c7-47f2-899e-bbb1d0cbea92"
-					(reference "#PWR051")
+					(reference "#PWR037")
 					(unit 1)
 				)
@@
 		(dnp no)
 		(fields_autoplaced yes)
-		(property "Reference" "JP9"
+		(property "Reference" "JP13"
 			(at 59.69 20.32 0)
 			(effects
@@
 			(project "bias-supply"
 				(path "/f3205b63-fc57-4ea3-95d4-2a447f249c30/2946e9e0-97c7-47f2-899e-bbb1d0cbea92"
-					(reference "JP9")
+					(reference "JP13")
 					(unit 1)
 				)
@@
 		(on_board yes)
 		(dnp no)
-		(property "Reference" "#PWR049"
+		(property "Reference" "#PWR035"
 			(at 49.53 36.83 0)
 			(effects
@@
 			(project "bias-supply"
 				(path "/f3205b63-fc57-4ea3-95d4-2a447f249c30/2946e9e0-97c7-47f2-899e-bbb1d0cbea92"
-					(reference "#PWR049")
+					(reference "#PWR035")
 					(unit 1)
 				)
@@
 		(on_board yes)
 		(dnp no)
-		(property "Reference" "#PWR053"
+		(property "Reference" "#PWR039"
 			(at 69.85 36.83 0)
 			(effects
@@
 			(project "bias-supply"
 				(path "/f3205b63-fc57-4ea3-95d4-2a447f249c30/2946e9e0-97c7-47f2-899e-bbb1d0cbea92"
-					(reference "#PWR053")
+					(reference "#PWR039")
 					(unit 1)
 				)
@@
 		(on_board yes)
 		(dnp no)
-		(property "Reference" "#PWR050"
+		(property "Reference" "#PWR036"
 			(at 49.53 53.34 0)
 			(effects
@@
 			(project "bias-supply"
 				(path "/f3205b63-fc57-4ea3-95d4-2a447f249c30/2946e9e0-97c7-47f2-899e-bbb1d0cbea92"
-					(reference "#PWR050")
+					(reference "#PWR036")
 					(unit 1)
 				)
@@
 		(dnp no)
 		(fields_autoplaced yes)
-		(property "Reference" "JP7"
+		(property "Reference" "JP9"
 			(at 34.29 20.32 0)
 			(effects
@@
 			(project ""
 				(path "/f3205b63-fc57-4ea3-95d4-2a447f249c30/2946e9e0-97c7-47f2-899e-bbb1d0cbea92"
-					(reference "JP7")
+					(reference "JP9")
 					(unit 1)
 				)
@@
 		(on_board yes)
 		(dnp no)
-		(property "Reference" "#PWR05"
+		(property "Reference" "#PWR026"
 			(at 24.13 26.67 0)
 			(effects
@@
 			(project "bias-supply"
 				(path "/f3205b63-fc57-4ea3-95d4-2a447f249c30/2946e9e0-97c7-47f2-899e-bbb1d0cbea92"
-					(reference "#PWR05")
+					(reference "#PWR026")
 					(unit 1)
 				)
@@
 		(on_board yes)
 		(dnp no)
-		(property "Reference" "#PWR052"
+		(property "Reference" "#PWR038"
 			(at 69.85 26.67 0)
 			(effects
@@
 			(project "bias-supply"
 				(path "/f3205b63-fc57-4ea3-95d4-2a447f249c30/2946e9e0-97c7-47f2-899e-bbb1d0cbea92"
-					(reference "#PWR052")
+					(reference "#PWR038")
 					(unit 1)
 				)
@@
 		(on_board yes)
 		(dnp no)
-		(property "Reference" "#PWR039"
+		(property "Reference" "#PWR028"
 			(at 24.13 53.34 0)
 			(effects
@@
 			(project "bias-supply"
 				(path "/f3205b63-fc57-4ea3-95d4-2a447f249c30/2946e9e0-97c7-47f2-899e-bbb1d0cbea92"
-					(reference "#PWR039")
+					(reference "#PWR028")
 					(unit 1)
 				)
@@
 		(on_board yes)
 		(dnp no)
-		(property "Reference" "#PWR047"
+		(property "Reference" "#PWR033"
 			(at 44.45 63.5 0)
 			(effects
@@
 			(project "bias-supply"
 				(path "/f3205b63-fc57-4ea3-95d4-2a447f249c30/2946e9e0-97c7-47f2-899e-bbb1d0cbea92"
-					(reference "#PWR047")
+					(reference "#PWR033")
 					(unit 1)
 				)
@@
 		(on_board yes)
 		(dnp no)
-		(property "Reference" "#PWR038"
+		(property "Reference" "#PWR027"
 			(at 24.13 36.83 0)
 			(effects
@@
 			(project "bias-supply"
 				(path "/f3205b63-fc57-4ea3-95d4-2a447f249c30/2946e9e0-97c7-47f2-899e-bbb1d0cbea92"
-					(reference "#PWR038")
+					(reference "#PWR027")
 					(unit 1)
 				)
@@
 		(dnp no)
 		(fields_autoplaced yes)
-		(property "Reference" "JP14"
+		(property "Reference" "JP16"
 			(at 59.69 57.15 0)
 			(effects
@@
 			(project "bias-supply"
 				(path "/f3205b63-fc57-4ea3-95d4-2a447f249c30/2946e9e0-97c7-47f2-899e-bbb1d0cbea92"
-					(reference "JP14")
+					(reference "JP16")
 					(unit 1)
 				)
@@
 		(dnp no)
 		(fields_autoplaced yes)
-		(property "Reference" "JP13"
+		(property "Reference" "JP15"
 			(at 59.69 46.99 0)
 			(effects
@@
 			(project "bias-supply"
 				(path "/f3205b63-fc57-4ea3-95d4-2a447f249c30/2946e9e0-97c7-47f2-899e-bbb1d0cbea92"
-					(reference "JP13")
+					(reference "JP15")
 					(unit 1)
 				)
@@
 		(on_board yes)
 		(dnp no)
-		(property "Reference" "#PWR040"
+		(property "Reference" "#PWR029"
 			(at 24.13 63.5 0)
 			(effects
@@
 			(project "bias-supply"
 				(path "/f3205b63-fc57-4ea3-95d4-2a447f249c30/2946e9e0-97c7-47f2-899e-bbb1d0cbea92"
-					(reference "#PWR040")
+					(reference "#PWR029")
 					(unit 1)
 				)
@@
 		(on_board yes)
 		(dnp no)
-		(property "Reference" "#PWR044"
+		(property "Reference" "#PWR030"
 			(at 44.45 26.67 0)
 			(effects
@@
 			(project "bias-supply"
 				(path "/f3205b63-fc57-4ea3-95d4-2a447f249c30/2946e9e0-97c7-47f2-899e-bbb1d0cbea92"
-					(reference "#PWR044")
+					(reference "#PWR030")
 					(unit 1)
 				)
@@
 		(on_board yes)
 		(dnp no)
-		(property "Reference" "#PWR048"
+		(property "Reference" "#PWR034"
 			(at 49.53 26.67 0)
 			(effects
@@
 			(project "bias-supply"
 				(path "/f3205b63-fc57-4ea3-95d4-2a447f249c30/2946e9e0-97c7-47f2-899e-bbb1d0cbea92"
-					(reference "#PWR048")
-					(unit 1)
-				)
+					(reference "#PWR034")
+					(unit 1)
+				)

Commit message: Bubba V2.1
Parts:
- added JP13: ~, Resistor_SMD:R_1206_3216Metric, symbol Jumper:SolderJumper_2_Open
- renumbered JP13 to JP14, JP14 to JP15, JP15 to JP16, JP16 to JP17
Connections:
- net GND: now also JP13.1 (A), JP13.2 (B)
Other:
- note added: "+V GND to +3V3 reg. GND"
