File: bias-supply/power-amp.kicad_sch (KiCad schematic)
At the start: 9 parts, among them U2 TCA0372BDWR2G

Commit message: Updated notes
Other:
- title: Power amp with controllable gain -> Power amp
Changed lines of the file:
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@@
 	(paper "A4")
 	(title_block
-		(title "Power amp with controllable gain")
-		(date "2025-03-28")
-		(rev "1.0")
+		(title "Power amp")
+		(date "2025-06-12")
+		(rev "2.0")
 	)
 	(rectangle

Commit message: Add fuses; change to coax; fixed I2C gnd
Parts:
- renumbered C17 to C15, C15 to C16, C16 to C17, R8 to R15, R9 to R16, R7 to R17
Changed lines of the file:
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@@
 		(on_board yes)
 		(dnp no)
-		(property "Reference" "R9"
+		(property "Reference" "R16"
 			(at 113.03 74.9299 0)
 			(effects
@@
 			(project "bias-supply"
 				(path "/f3205b63-fc57-4ea3-95d4-2a447f249c30/8e2238c6-8ba6-47bd-8ae1-ac4c58bee3fb"
-					(reference "R9")
+					(reference "R16")
 					(unit 1)
 				)
@@
 		(on_board yes)
 		(dnp no)
-		(property "Reference" "#PWR015"
+		(property "Reference" "#PWR018"
 			(at 185.42 73.66 0)
 			(effects
@@
 			(project "bias-supply"
 				(path "/f3205b63-fc57-4ea3-95d4-2a447f249c30/8e2238c6-8ba6-47bd-8ae1-ac4c58bee3fb"
-					(reference "#PWR015")
+					(reference "#PWR018")
 					(unit 1)
 				)
@@
 		(on_board yes)
 		(dnp no)
-		(property "Reference" "#PWR018"
+		(property "Reference" "#PWR017"
 			(at 120.65 64.77 0)
 			(effects
@@
 			(project "bias-supply"
 				(path "/f3205b63-fc57-4ea3-95d4-2a447f249c30/8e2238c6-8ba6-47bd-8ae1-ac4c58bee3fb"
-					(reference "#PWR018")
+					(reference "#PWR017")
 					(unit 1)
 				)
@@
 		(on_board yes)
 		(dnp no)
-		(property "Reference" "C17"
+		(property "Reference" "C15"
 			(at 128.27 50.8 90)
 			(effects
@@
 			(project "bias-supply"
 				(path "/f3205b63-fc57-4ea3-95d4-2a447f249c30/8e2238c6-8ba6-47bd-8ae1-ac4c58bee3fb"
-					(reference "C17")
+					(reference "C15")
 					(unit 1)
 				)
@@
 		(on_board yes)
 		(dnp no)
-		(property "Reference" "C16"
+		(property "Reference" "C17"
 			(at 182.88 69.85 90)
 			(effects
@@
 			(project "bias-supply"
 				(path "/f3205b63-fc57-4ea3-95d4-2a447f249c30/8e2238c6-8ba6-47bd-8ae1-ac4c58bee3fb"
-					(reference "C16")
+					(reference "C17")
 					(unit 1)
 				)
@@
 		(on_board yes)
 		(dnp no)
-		(property "Reference" "#PWR028"
+		(property "Reference" "#PWR016"
 			(at 119.38 55.88 0)
 			(effects
@@
 			(project "bias-supply"
 				(path "/f3205b63-fc57-4ea3-95d4-2a447f249c30/8e2238c6-8ba6-47bd-8ae1-ac4c58bee3fb"
-					(reference "#PWR028")
+					(reference "#PWR016")
 					(unit 1)
 				)
@@
 		(dnp no)
 		(fields_autoplaced yes)
-		(property "Reference" "#PWR016"
+		(property "Reference" "#PWR015"
 			(at 115.57 85.09 0)
 			(effects
@@
 			(project "bias-supply"
 				(path "/f3205b63-fc57-4ea3-95d4-2a447f249c30/8e2238c6-8ba6-47bd-8ae1-ac4c58bee3fb"
-					(reference "#PWR016")
+					(reference "#PWR015")
 					(unit 1)
 				)
@@
 		(on_board yes)
 		(dnp no)
-		(property "Reference" "R7"
+		(property "Reference" "R17"
 			(at 132.08 78.74 90)
 			(effects
@@
 			(project ""
 				(path "/f3205b63-fc57-4ea3-95d4-2a447f249c30/8e2238c6-8ba6-47bd-8ae1-ac4c58bee3fb"
-					(reference "R7")
+					(reference "R17")
 					(unit 1)
 				)
@@
 		(on_board yes)
 		(dnp no)
-		(property "Reference" "R8"
+		(property "Reference" "R15"
 			(at 113.03 63.4999 0)
 			(effects
@@
 			(project ""
 				(path "/f3205b63-fc57-4ea3-95d4-2a447f249c30/8e2238c6-8ba6-47bd-8ae1-ac4c58bee3fb"
-					(reference "R8")
+					(reference "R15")
 					(unit 1)
 				)
@@
 		(on_board yes)
 		(dnp no)
-		(property "Reference" "C15"
+		(property "Reference" "C16"
 			(at 129.54 69.85 90)
 			(effects
@@
 			(project "bias-supply"
 				(path "/f3205b63-fc57-4ea3-95d4-2a447f249c30/8e2238c6-8ba6-47bd-8ae1-ac4c58bee3fb"
-					(reference "C15")
+					(reference "C16")
 					(unit 1)
 				)

Commit message: Bubba V2.1
Parts:
- RV1: now not fitted; now left out of the parts list
- SIN2: now left out of the parts list
Changed lines of the file:
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@@
 	(title_block
 		(title "Power amp")
-		(date "2025-06-12")
-		(rev "2.0")
+		(date "2026-03-05")
+		(rev "2.1")
 	)
 	(rectangle
@@
 			)
 		)
-		(property "Datasheet" "~"
+		(property "Datasheet" "https://yageogroup.com/content/datasheet/asset/file/PYU-RC_GROUP_51_ROHS_L"
 			(at 115.57 76.2 0)
 			(effects
@@
 			)
 		)
-		(property "Description" "Resistor, small symbol"
+		(property "Description" "RC1206FR-07100KL"
 			(at 115.57 76.2 0)
 			(effects
@@
 			)
 		)
-		(property "Description" "ON SEMICONDUCTOR - TCA0372BDWR2G - OP-AMP, DUAL, 1.4MHZ, 1.4V/US, WSOIC-16"
+		(property "Description" "TCA0372BDWR2G"
 			(at 135.89 55.88 0)
 			(effects
@@
 		(unit 1)
 		(exclude_from_sim no)
-		(in_bom yes)
+		(in_bom no)
 		(on_board yes)
-		(dnp no)
+		(dnp yes)
 		(property "Reference" "RV1"
 			(at 95.25 69.596 0)
@@
 			)
 		)
-		(property "Datasheet" "~"
+		(property "Datasheet" "https://search.murata.co.jp/Ceramy/image/img/A01X/G101/ENG/GRM3195C2A104GA01-01A.pdf"
 			(at 128.27 55.88 0)
 			(effects
@@
 			)
 		)
-		(property "Description" "Unpolarized capacitor, small symbol"
+		(property "Description" "GRM3195C2A104GA01D"
 			(at 128.27 55.88 0)
 			(effects
@@
 			)
 		)
-		(property "Datasheet" "~"
+		(property "Datasheet" "https://search.murata.co.jp/Ceramy/image/img/A01X/G101/ENG/GRM3195C2A104GA01-01A.pdf"
 			(at 182.88 64.77 0)
 			(effects
@@
 			)
 		)
-		(property "Description" "Unpolarized capacitor, small symbol"
+		(property "Description" "GRM3195C2A104GA01D"
 			(at 182.88 64.77 0)
 			(effects
@@
 			)
 		)
-		(property "Datasheet" "~"
+		(property "Datasheet" "https://yageogroup.com/content/datasheet/asset/file/PYU-RC_GROUP_51_ROHS_L"
 			(at 132.08 73.66 0)
 			(effects
@@
 			)
 		)
-		(property "Description" "Resistor, small symbol"
+		(property "Description" "RC1206FR-0710KL"
 			(at 132.08 73.66 0)
 			(effects
@@
 		(unit 1)
 		(exclude_from_sim no)
-		(in_bom yes)
+		(in_bom no)
 		(on_board yes)
 		(dnp no)
@@
 			)
 		)
-		(property "Datasheet" "~"
+		(property "Datasheet" "https://industrial.panasonic.com/cdbs/www-data/pdf/RDM0000/AOA0000C307.pdf"
 			(at 115.57 64.77 0)
 			(effects
@@
 			)
 		)
-		(property "Description" "Resistor, small symbol"
+		(property "Description" "ERA-8AEB3832V"
 			(at 115.57 64.77 0)
 			(effects
@@
 			)
 		)
-		(property "Datasheet" "~"
+		(property "Datasheet" "https://search.murata.co.jp/Ceramy/image/img/A01X/G101/ENG/GRM3195C2A104GA01-01A.pdf"
 			(at 129.54 64.77 0)
 			(effects
@@
 			)
 		)
-		(property "Description" "Unpolarized capacitor, small symbol"
+		(property "Description" "GRM3195C2A104GA01D"
 			(at 129.54 64.77 0)
 			(effects
