File: lvps-swri/IMPISH Power Supply.kicad_pcb (KiCad board)
At the start: 4 copper layers, 90 x 90 mm, 68 parts, among them J1 Battery +, J2 Battery +, J3 Battery -, J4 Battery -, J5 BCS-117-L-D-TE, U1 PXG-M15-24WS05, U2 CCG30-24-12S, U3 PXC-M03-24WD15-A, U4 PXC-M03-24WS05-A, U5 PXG-M15-24WD05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

Commit message: Power board updates (#7)
* toggles adapter board

The SwRI toggle output is in the wrong direction,
so we are adding an additional PCB to point the power
towards the side of the EPS box. We can route it with
cables and connectors instead of using the board-to-board
style interface.

* toggles adapter: cleanup

* toggles adapter: via stitching

* swri toggles: start one ground

* swri toggles: single ground pre stitching

* swri toggles: via stitching for gnd

* swri toggles: fix DRC and ERC errors

* swri lvps main: two layer board

* swri lvps main: fix cap models
Parts:
- removed C12, C16, C20, C26, C31, C6: .01uF, Capacitor_SMD:C_0805_2012Metric_Pad1.18x1.45mm_HandSolder
- removed JP1, JP2, JP3, JP4, JP5: ~, Jumper:SolderJumper-2_P1.3mm_Open_Pad1.0x1.5mm
- removed R1, R2, R3: 0, Resistor_SMD:R_0805_2012Metric_Pad1.20x1.40mm_HandSolder
- removed R4, R5, R6, R7: DNI, Resistor_SMD:R_0805_2012Metric_Pad1.20x1.40mm_HandSolder
- C1, C21: footprint IMPISH Library:CAPC4520X150N -> IMPISH Library:CAP_DE2B3SA101KN3AY02F
- moved G*** 2.65 mm to (205.4, 143.0)
- moved C21 0.73 mm to (179.2, 141.8)
Connections:
- J5 pad 03: GND1 -> GND
- J5 pad 04: GND1 -> GND
- J5 pad 07: Cremat GND -> GND
- J5 pad 08: Cremat GND -> GND
- J5 pad 11: Bridgeport GND -> GND
- J5 pad 12: Bridgeport GND -> GND
- J5 pad 17: Bias GND -> GND
- J5 pad 18: Bias GND -> GND
- J5 pad 21: Heater GND -> GND
- J5 pad 22: Heater GND -> GND
- J5 pad 27: SiPM GND -> GND
- J5 pad 28: SiPM GND -> GND
- U1 pad 3: Net-(U1-REMOTE_ON/OFF) -> GND
- U1 pad 5: GND1 -> GND
- U1 pad 6: Net-(U1-TRIM) -> unconnected-(U1-TRIM-Pad6)
- U2 pad 3: Net-(U2-RC) -> GND
- U2 pad 5: Net-(U2-TRM) -> unconnected-(U2-TRM-Pad5)
- U2 pad 6: Heater GND -> GND
- U3 pad 11: Bias GND -> GND
- U4 pad 12: Bridgeport GND -> GND
- U5 pad 3: Net-(U5-REMOTE_ON/OFF) -> GND
- U5 pad 5: SiPM GND -> GND
- U6 pad 16: Cremat GND -> GND
- U6 pad 9: Cremat GND -> GND
Routing:
- net GND1: track 135.3 -> 0.00 mm
- net Cremat GND: track 92.3 -> 0.00 mm
- net GND: track 110.7 -> 18.7 mm, vias 77 -> 0
- net Bias GND: track 76.5 -> 0.00 mm
- net SiPM GND: track 61.9 -> 0.00 mm
- net Heater GND: track 25.8 -> 0.00 mm
- net Bridgeport GND: track 22.8 -> 0.00 mm
- net Net-(U2-TRM): track 10.9 -> 0.00 mm
- net Net-(U1-TRIM): track 10.7 -> 0.00 mm
- net CM4 +5V: track 53.4 -> 60.8 mm
- net Heater 12V: track 36.1 -> 31.4 mm
- net Net-(U1-REMOTE_ON/OFF): track 4.22 -> 0.00 mm
- net Net-(U5-REMOTE_ON/OFF): track 4.03 -> 0.00 mm
- net Net-(U2-RC): track 3.20 -> 0.00 mm
- net CHASSIS: track 16.5 -> 13.3 mm, vias 981 -> 979
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- added copper zone on B.Cu, net GND
- removed copper zone on In1.Cu, net GND
Other:
- copper layers 4 -> 2
- board text added: "and friends"

Commit message: update main PSU: soldermask near edge
Routing:
- net CHASSIS: vias 979 -> 972
Other:
- board text removed: "0"
- board text removed: "0 mm"
- board text removed: "0.0000 mm / 0.0000 mm"
- board text removed: "0.01 mm"
- board text removed: "0.02"
- board text removed: "0.07 mm"
- board text removed: "0.1 mm"
- board text removed: "0.3000 mm"
- board text removed: "1"
- board text removed: "1.07 mm"
- board text removed: "1.5700 mm"
- board text removed: "3.3"
- board text removed: "4"
- board text removed: "4.5"
- board text removed: "90.0000 mm x 90.0000 mm"
- board text removed: "B.Cu"
- board text removed: "B.Mask"
- board text removed: "B.Paste"
- board text removed: "B.Silkscreen"
- board text removed: "BOARD CHARACTERISTICS"
- board text removed: "Board Thickness:"
- board text removed: "Board overall dimensions:"
- board text removed: "Bottom Silk Screen"
- board text removed: "Bottom Solder Mask"
- board text removed: "Bottom Solder Paste"
- board text removed: "Castellated pads:"
- board text removed: "Color"
- board text removed: "Copper Finish:"
- board text removed: "Copper Layer Count:"
- board text removed: "Dielectric"
- board text removed: "Edge card connectors:"
- board text removed: "Epsilon R"
- board text removed: "F.Cu"
- board text removed: "F.Mask"
- board text removed: "F.Paste"
- board text removed: "F.Silkscreen"
- board text removed: "FR4"
- board text removed: "Impedance Control:"
- board text removed: "In1.Cu"
- board text removed: "In2.Cu"
- board text removed: "Layer Name"
- board text removed: "Loss Tangent"
- board text removed: "Material"
- board text removed: "Min hole diameter:"
- board text removed: "Min track/spacing:"
- board text removed: "No"
- board text removed: "None"
- board text removed: "Not specified"
- board text removed: "Plated Board Edge:"
- board text removed: "Thickness (mm)"
- board text removed: "Top Silk Screen"
- board text removed: "Top Solder Mask"
- board text removed: "Top Solder Paste"
- board text removed: "Type"
- board text removed: "copper"
- board text removed: "core"
- board text removed: "prepreg"
